File: Projects/Fresu/BLDC Motor Controller/Design/rev01/rev01_1/BLDC_Motor Controller/MCU.kicad_sch (KiCad schematic)
At the start: 0 parts

Commit message: Update 5
nearly completed MCU schematic, PDF version is wrong so waiting for it to be fixed
Parts:
- added C1: C, symbol Device:C
- added C10, C9: 2u2, symbol Device:C
- added C11, C15, C16: 100n, symbol Device:C
- added C12: 1u, symbol Device:C
- added C13, C14: 10p, symbol Device:C
- added C2, C3, C4, C5, C6, C7, C8: 100nF, symbol Device:C
- added D1, D6: LED_G, symbol Device:LED
- added D2: LED_R, symbol Device:LED
- added D3, D4: BAT60A, Diode_SMD:D_SOD-323, symbol Diode:BAT60A
- added D5: SD05_SOD323, Diode_SMD:D_SOD-323, symbol Diode:SD05_SOD323
- added FB1: FerriteBead, symbol Device:FerriteBead
- added J1: Conn_01x06, symbol Connector_Generic:Conn_01x06
- added J2: Conn_01x03, symbol Connector_Generic:Conn_01x03
- added J3: Conn_01x08, symbol Connector_Generic:Conn_01x08
- added R1: 100R, symbol Device:R
- added R2, R3: 0R, symbol Device:R
- added R4, R5, R6: 1k, symbol Device:R
- added R7, R8: 2k2, symbol Device:R
- added SW1: SW_DIP_x01, symbol Switch:SW_DIP_x01
- added TH1: 10K, symbol Device:Thermistor_NTC
- added U1: STM32F405RGTx, Package_QFP:LQFP-64_10x10mm_P0.5mm, symbol MCU_ST_STM32F4:STM32F405RGTx
- added Y1: 8MHz, symbol Device:Crystal
Connections:
- new net: D2.2 (A), R5.1
- new net: D6.2 (A), R6.1
- new net: D1.2 (A), R4.1
- new net: J2.3 (Pin_3), R7.1
- new net +3V3: C1.1, C16.1, C2.1, C3.1, C4.1, C5.1, C6.1, C7.1, FB1.2, J1.1 (Pin_1), R6.2, TH1.1, U1.19 (VDD), U1.32 (VDD), U1.48 (VDD), U1.64 (VDD)
- new net +3V3_A: C11.1, C12.1, FB1.1, U1.13 (VDDA)
- new net +5V: J2.1 (Pin_1), J3.1 (Pin_1)
- new net ADC_TEMP: R8.1, TH1.2, U1.17 (PA3)
- new net AN_IN: U1.10 (PC2)
- new net BOOT0_P: R1.2, U1.60 (BOOT0)
- new net BR_S01: U1.27 (PB1)
- new net BR_S02: U1.26 (PB0)
- new net CAN_RX: U1.61 (PB8)
- new net CAN_TX: U1.62 (PB9)
- new net DC_CAL: U1.33 (PB12)
- new net EN_GATE: U1.51 (PC10)
- new net FAULT: U1.53 (PC12)
- new net GND: C1.2, C10.2, C11.2, C12.2, C13.2, C14.2, C15.2, C16.2, C2.2, C3.2, C4.2, C5.2, C6.2, C7.2, C8.2, C9.2, D1.1 (K), D2.1 (K), D6.1 (K), J1.3 (Pin_3), J2.2 (Pin_2), R1.1, R8.2, SW1.1, U1.12 (VSSA), U1.18 (VSS), U1.63 (VSS)
- new net H1: U1.43 (PA10)
- new net H2: U1.42 (PA9)
- new net H3: U1.41 (PA8)
- new net HALL_1_OUT: U1.58 (PB6)
- new net HALL_2_OUT: U1.59 (PB7)
- new net HALL_3_OUT: U1.52 (PC11)
- new net L1: U1.36 (PB15)
- new net L2: U1.35 (PB14)
- new net L3: U1.34 (PB13)
- new net LED_GREEN: R4.2, U1.24 (PC4)
- new net LED_RED: R5.2, U1.25 (PC5)
- new net MISO_ADC_EXT: U1.22 (PA6)
- new net NRST: C8.1, J1.5 (Pin_5), SW1.2, U1.7 (NRST)
- new net PH_0: C13.1, R2.1, Y1.2
- new net PH_0_P: R2.2, U1.5 (PH0)
- new net PH_1: C14.1, R3.1, Y1.1
- new net PH_1_P: R3.2, U1.6 (PH1)
- new net RX_SCI_MOSI: U1.23 (PA7)
- new net RX_SDA_NSS: U1.30 (PB11), U1.37 (PC6)
- new net SCK_ADC_EXT: U1.21 (PA5)
- new net SENS1: U1.14 (PA0), U1.16 (PA2)
- new net SENS2: U1.15 (PA1)
- new net SERVO: C15.1, R7.2, U1.57 (PB5)
- new net SWCLK: J1.2 (Pin_2), U1.49 (PA14)
- new net SWDIO: J1.4 (Pin_4), U1.46 (PA13)
- new net TEMP_MOTOR: U1.8 (PC0)
- new net TX_SCI_MOSI: U1.29 (PB10)
- new net TX_SCL_MOSI: U1.38 (PC7)
- new net TX_SDA_NSS: U1.20 (PA4)
- new net USB_DM: U1.44 (PA11)
- new net USB_DP: U1.45 (PA12)
- new net VCAP_1: C9.1, U1.31 (VCAP_1)
- new net VCAP_2: C10.1, U1.47 (VCAP_2)
- no-connect marks 0 -> 13
Other:
- note added: "COMMUNICATION"
- note added: "FEEDBACK MCU"
- note added: "HALL ENCODER"
- note added: "INPUT"
- note added: "NTC THERMISTOR"
- note added: "PROGRAMMING / DEBUG"
- note added: "SENSING"
- note added: "SERVO"
- note added: "SUBSTITUE WITH 100R IF USED AS SERVO OUTPUT"
- note added: "USB BUS"
- note added: "X50328MSB2GI"

Commit message: UPDATE 6
Completed MCU schematic Page
Parts:
- added C17: 100nF, symbol Device:C
- added R10: 2k2, symbol Device:R
- added R9: 39k, symbol Device:R
Connections:
- net GND: now also J3.8 (Pin_8), C17.2, R10.1
- net MISO_ADC_EXT: now also J3.7 (Pin_7)
- net RX_SDA_NSS: now also J3.5 (Pin_5)
- net SCK_ADC_EXT: now also J3.4 (Pin_4)
- net TX_SCL_MOSI: now also J3.6 (Pin_6)
- new net: C17.1, R10.2, R9.1
- new net +VDC: R9.2
Other:
- note added: "VOLTAGE DIVIDER"
- note added: "WHEN: VIN = 60 -> AN_IN = 3V204"

Commit message: Update 13
Added:
1) USB Schematic
2) footprints to all parts
Parts:
- removed SW1: SW_DIP_x01, symbol Switch:SW_DIP_x01
- added R56: 2k2, Resistor_SMD:R_0603_1608Metric_Pad0.98x0.95mm_HandSolder, symbol Device:R
- added SW2: PTS526SK15SMTR2LFS, DF_ESC_Footprint_Library:SW-SMD_4P-L5.2-W5.2-P3.70-LS6.4, symbol DF_ESC_Symbol_Library:PTS526SK15SMTR2LFS
- C1, C10, C11, C12, C13, C14, C15, C16, C17, C2, C3, C4, C5, C6, C7, C8, C9: footprint (none) -> Capacitor_SMD:C_0603_1608Metric
- D1, D2, D6: footprint (none) -> LED_SMD:LED_1206_3216Metric
- FB1: footprint (none) -> Inductor_SMD:L_0603_1608Metric_Pad1.05x0.95mm_HandSolder
- J1: footprint (none) -> DF_ESC_Footprint_Library:CONN-SMD_S6B-XH-SM4-TB-LF-SN
- J2: footprint (none) -> DF_ESC_Footprint_Library:CONN-SMD_XH-3AWB
- J3: footprint (none) -> DF_ESC_Footprint_Library:CONN-SMD_8P-P2.50_HX25003-8AWB
- R1, R10, R2, R3, R4, R5, R6, R7, R8, R9, TH1: footprint (none) -> Resistor_SMD:R_0603_1608Metric_Pad0.98x0.95mm_HandSolder
- Y1: footprint (none) -> DF_ESC_Footprint_Library:CRYSTAL-SMD_L5.0-W3.2
Connections:
- net GND: now also R56.1
- net NRST: now also SW2.3, SW2.4
- new net: R56.2, SW2.1, SW2.2
- no-connect marks 13 -> 19

Commit message: Update 15
Fixing some schematic errors

initial layout of larger component complete
Parts:
- removed C16: 100n, Capacitor_SMD:C_0603_1608Metric, symbol Device:C
- removed R8: 2k2, Resistor_SMD:R_0603_1608Metric_Pad0.98x0.95mm_HandSolder, symbol Device:R
- removed TH1: 10K, Resistor_SMD:R_0603_1608Metric_Pad0.98x0.95mm_HandSolder, symbol Device:Thermistor_NTC
- added D15: BAT60A, Diode_SMD:D_SOD-323, symbol Diode:BAT60A
- renumbered C9 to C10, C8 to C11, C17 to C12, C10 to C13, C11 to C14, C12 to C15, C15 to C16, C13 to C8, C14 to C9, D6 to D1, D5 to D2, D1 to D5, D2 to D6, J3 to J1, J1 to J2, J2 to J3, R6 to R1, R7 to R10, R4 to R2, R56 to R3, R5 to R4, R2 to R5, R3 to R6, R9 to R7, R10 to R8, R1 to R9, SW2 to SW1
Connections:
- net RX_SCI_MOSI is gone; now on net TX_SCI_MOSI: U1.23 (PA7)
- net TX_SDA_NSS is gone; now on net RX_SDA_NSS: U1.20 (PA4)
- net USB_DM is gone; now on net USB_N: U1.44 (PA11)
- net USB_DP is gone; now on net USB_P: U1.45 (PA12)
- net +3V3: now also D4.1 (K), U1.1 (VBAT), D15.1 (K); no longer J2.1 (Pin_1)
- net +5V: now also D3.1 (K); no longer J1.1 (Pin_1)
- net GND: now also D2.1 (A1), J1.3 (Pin_3), J2.5 (Pin_5)
- net NRST: now also J2.6 (Pin_6); no longer J2.5 (Pin_5)
- net SENS1: no longer U1.14 (PA0)
- net SWCLK: now also J2.4 (Pin_4); no longer J2.2 (Pin_2)
- net SWDIO: now also J2.2 (Pin_2); no longer J2.4 (Pin_4)
- net at D2.2 (A2): now also D3.2 (A), J1.1 (Pin_1)
- net at D4.2 (A): now also J1.2 (Pin_2)
- net MISO_ADC_EXT renamed MISO_ADC_EXT2
- new net: D15.2 (A), J2.1 (Pin_1)
- new net SENS3: U1.14 (PA0)
- no-connect marks 19 -> 18
Other:
- note added: "INPUT PORTS"
- note removed: "NTC THERMISTOR"
- moved on the sheet: C12, D2, D3, D4, R7, R8

Commit message: Update 16
Almost finished placing all the components on the board as rough placement
Parts:
- removed C12: 100nF, Capacitor_SMD:C_0603_1608Metric, symbol Device:C
- removed D1: LED_G, LED_SMD:LED_1206_3216Metric, symbol Device:LED
- removed R1: 1k, Resistor_SMD:R_0603_1608Metric_Pad0.98x0.95mm_HandSolder, symbol Device:R
- removed R7: 39k, Resistor_SMD:R_0603_1608Metric_Pad0.98x0.95mm_HandSolder, symbol Device:R
- removed R8: 2k2, Resistor_SMD:R_0603_1608Metric_Pad0.98x0.95mm_HandSolder, symbol Device:R
Other:
- note removed: "VOLTAGE DIVIDER"
- note removed: "WHEN: VIN = 60 -> AN_IN = 3V204"

Commit message: Update 17
Started laying out the driver and the main FET power polygons
Parts:
- C1: value C -> 10u
Changed lines of the file:
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@@
       (effects (font (size 1.27 1.27)) (justify left))
     )
-    (property "Value" "C" (at 29.21 30.48 0)
+    (property "Value" "10u" (at 29.21 30.48 0)
       (effects (font (size 1.27 1.27)) (justify left))
     )

Commit message: Update 18
almost done routing driver chip and MCU (first pass)
Connections:
- net TX_SCI_MOSI is gone; now on net TX_SCL_MOSI: U1.23 (PA7), U1.29 (PB10)
Changed lines of the file:
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@@
     (effects (font (size 1.27 1.27)) (justify left bottom))
   )
-  (label "TX_SCI_MOSI" (at 181.61 121.92 0) (fields_autoplaced)
+  (label "TX_SCL_MOSI" (at 181.61 121.92 0) (fields_autoplaced)
     (effects (font (size 1.27 1.27)) (justify left bottom))
   )
@@
     (effects (font (size 1.27 1.27) bold) (justify right bottom))
   )
-  (label "TX_SCI_MOSI" (at 181.61 68.58 0) (fields_autoplaced)
-    (effects (font (size 1.27 1.27)) (justify left bottom))
-  )
   (label "PH_1_P" (at 128.27 85.09 0) (fields_autoplaced)
     (effects (font (size 1.27 1.27) bold) (justify left bottom))
@@
     (effects (font (size 1.27 1.27)) (justify left bottom))
   )
+  (label "TX_SCL_MOSI" (at 181.61 68.58 0) (fields_autoplaced)
+    (effects (font (size 1.27 1.27)) (justify left bottom))
+  )

Commit message: Update 20
First layout completed, all tracks laid
Parts:
- removed C6: 100nF, Capacitor_SMD:C_0603_1608Metric, symbol Device:C
Connections:
- net CAN_RX renamed CAN-
- net CAN_TX renamed CAN+
Changed lines of the file:
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@@
   (junction (at 72.39 24.13) (diameter 0) (color 0 0 0 0)
   )
-  (junction (at 78.74 24.13) (diameter 0) (color 0 0 0 0)
-  )
   (junction (at 123.19 71.12) (diameter 0) (color 0 0 0 0)
   )
   (junction (at 189.23 35.56) (diameter 0) (color 0 0 0 0)
-  )
-  (junction (at 78.74 35.56) (diameter 0) (color 0 0 0 0)
   )
   (junction (at 53.34 35.56) (diameter 0) (color 0 0 0 0)
@@
     (stroke (width 0) (type default))
   )
-  (wire (pts (xy 72.39 35.56) (xy 78.74 35.56))
-    (stroke (width 0) (type default))
-  )
   (wire (pts (xy 72.39 35.56) (xy 72.39 33.02))
     (stroke (width 0) (type default))
@@
     (stroke (width 0) (type default))
   )
-  (wire (pts (xy 78.74 24.13) (xy 85.09 24.13))
-    (stroke (width 0) (type default))
-  )
   (polyline (pts (xy 13.97 93.98) (xy 13.97 77.47))
     (stroke (width 0.5) (type default))
@@
     (stroke (width 0) (type default))
   )
-  (wire (pts (xy 72.39 24.13) (xy 78.74 24.13))
+  (wire (pts (xy 72.39 24.13) (xy 85.09 24.13))
     (stroke (width 0) (type default))
   )
@@
     (stroke (width 0.5) (type default))
   )
-  (wire (pts (xy 78.74 25.4) (xy 78.74 24.13))
-    (stroke (width 0) (type default))
-  )
   (wire (pts (xy 97.79 33.02) (xy 97.79 30.48))
     (stroke (width 0) (type default))
@@
     (stroke (width 0) (type default))
   )
-  (wire (pts (xy 78.74 35.56) (xy 85.09 35.56))
+  (wire (pts (xy 72.39 35.56) (xy 85.09 35.56))
     (stroke (width 0) (type default))
   )
@@
     (stroke (width 0.5) (type default))
   )
-  (wire (pts (xy 78.74 35.56) (xy 78.74 33.02))
-    (stroke (width 0) (type default))
-  )
   (wire (pts (xy 261.62 142.24) (xy 251.46 142.24))
     (stroke (width 0) (type default))
@@
     (effects (font (size 1.27 1.27)) (justify left bottom))
   )
-  (label "CAN_RX" (at 196.85 158.75 0) (fields_autoplaced)
-    (effects (font (size 1.27 1.27) bold) (justify left bottom))
-  )
   (label "NRST" (at 128.27 35.56 0) (fields_autoplaced)
     (effects (font (size 1.27 1.27) (thickness 0.254) bold) (justify left bottom))
@@
     (effects (font (size 1.27 1.27) bold) (justify right bottom))
   )
+  (label "CAN-" (at 196.85 158.75 0) (fields_autoplaced)
+    (effects (font (size 1.27 1.27) bold) (justify left bottom))
+  )
   (label "SWCLK" (at 250.19 102.87 0) (fields_autoplaced)
     (effects (font (size 1.27 1.27)) (justify left bottom))
@@
     (effects (font (size 1.27 1.27)) (justify left bottom))
   )
+  (label "CAN+" (at 196.85 156.21 0) (fields_autoplaced)
+    (effects (font (size 1.27 1.27) bold) (justify left bottom))
+  )
   (label "TX_SCL_MOSI" (at 181.61 121.92 0) (fields_autoplaced)
     (effects (font (size 1.27 1.27)) (justify left bottom))
@@
     (effects (font (size 1.27 1.27)) (justify left bottom))
   )
-  (label "CAN_TX" (at 196.85 156.21 0) (fields_autoplaced)
-    (effects (font (size 1.27 1.27) bold) (justify left bottom))
-  )
   (label "USB_N" (at 181.61 78.74 0) (fields_autoplaced)
     (effects (font (size 1.27 1.27)) (justify left bottom))
@@
     (effects (font (size 1.27 1.27) (thickness 0.254) bold) (justify left bottom))
   )
+  (label "CAN-" (at 181.61 116.84 0) (fields_autoplaced)
+    (effects (font (size 1.27 1.27) bold) (justify left bottom))
+  )
   (label "SENS3" (at 45.72 140.97 180) (fields_autoplaced)
     (effects (font (size 1.27 1.27) bold) (justify right bottom))
@@
     (effects (font (size 1.27 1.27)) (justify left bottom))
   )
+  (label "CAN+" (at 181.61 119.38 0) (fields_autoplaced)
+    (effects (font (size 1.27 1.27) bold) (justify left bottom))
+  )
   (label "L3" (at 260.35 58.42 0) (fields_autoplaced)
     (effects (font (size 1.27 1.27) bold) (justify left bottom))
@@
     (effects (font (size 1.27 1.27)) (justify left bottom))
   )
-  (label "CAN_RX" (at 181.61 116.84 0) (fields_autoplaced)
-    (effects (font (size 1.27 1.27)) (justify left bottom))
-  )
   (label "SENS1" (at 45.72 151.13 180) (fields_autoplaced)
     (effects (font (size 1.27 1.27) bold) (justify right bottom))
@@
   (label "L1" (at 260.35 45.72 0) (fields_autoplaced)
     (effects (font (size 1.27 1.27) bold) (justify left bottom))
-  )
-  (label "CAN_TX" (at 181.61 119.38 0) (fields_autoplaced)
-    (effects (font (size 1.27 1.27)) (justify left bottom))
   )
   (label "PH_0_P" (at 128.27 82.55 0) (fields_autoplaced)
@@
     )
   )
-  (global_label "CAN_TX" (shape input) (at 218.44 156.21 0) (fields_autoplaced)
+  (global_label "CAN+" (shape input) (at 218.44 156.21 0) (fields_autoplaced)
     (effects (font (size 1.27 1.27) bold) (justify left))
-    (property "Intersheetrefs" "${INTERSHEET_REFS}" (at 228.8301 156.21 0)
+    (property "Intersheetrefs" "${INTERSHEET_REFS}" (at 227.2578 156.21 0)
       (effects (font (size 1.27 1.27)) (justify left) hide)
     )
@@
     )
   )
-  (global_label "CAN_RX" (shape input) (at 218.44 158.75 0) (fields_autoplaced)
+  (global_label "CAN-" (shape input) (at 218.44 158.75 0) (fields_autoplaced)
     (effects (font (size 1.27 1.27) bold) (justify left))
-    (property "Intersheetrefs" "${INTERSHEET_REFS}" (at 229.1325 158.75 0)
+    (property "Intersheetrefs" "${INTERSHEET_REFS}" (at 227.2578 158.75 0)
       (effects (font (size 1.27 1.27)) (justify left) hide)
     )
@@
         )
       )
-    )
-  )
-  (symbol (lib_id "Device:C") (at 78.74 29.21 0) (unit 1)
-    (in_bom yes) (on_board yes) (dnp no)
-    (property "Reference" "C6" (at 80.01 26.67 0)
-      (effects (font (size 1.27 1.27)) (justify left))
-    )
-    (property "Value" "100nF" (at 69.85 29.21 0)
-      (effects (font (size 1.27 1.27)) (justify left) hide)
-    )
-    (property "Footprint" "Capacitor_SMD:C_0603_1608Metric" (at 79.7052 33.02 0)
-      (effects (font (size 1.27 1.27)) hide)
-    )
-    (property "Datasheet" "~" (at 78.74 29.21 0)
-      (effects (font (size 1.27 1.27)) hide)
-    )
-    (pin "2")
-    (pin "1")
-    (instances
-      (project "BLDC_Motor Controller"
-        (path "/e63e39d7-6ac0-4ffd-8aa3-1841a4541b55/6e5056e0-f286-40ca-8b4a-d506221b7bad"
-          (reference "C6") (unit 1)
-        )
-      )
