File: Projects/Fresu/BLDC Motor Controller/Design/rev01/rev01_1/BLDC_Motor Controller/MCU.kicad_sch (KiCad schematic)
At the start: 34 parts, among them J1 Conn_01x08, J2 Conn_01x06, J3 Conn_01x03, SW1 PTS526SK15SMTR2LFS, U1 STM32F405RGTx, Y1 8MHz

Commit message: Update 26
Matched DF's Designators to mine so I can use BOM as is

Updated MFR'ing files

Rev1 Ready for release
Parts:
- renumbered C4 to C10, C5 to C11, C8 to C12, C9 to C13, C7 to C14, C10 to C16, C11 to C17, C13 to C18, C14 to C19, C15 to C20, C16 to C21, C1 to C7, C2 to C8, C3 to C9, D6 to D10, D15 to D11, D2 to D5, D4 to D6, D3 to D8, D5 to D9, J1 to J2, J2 to J3, J3 to J4, R3 to R63, R2 to R7, R4 to R8, U1 to U2
Changed lines of the file:
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@@
 		(dnp no)
 		(fields_autoplaced yes)
-		(property "Reference" "D2"
-			(at 76.2 180.34 90)
+		(property "Reference" "D5"
+			(at 76.2 180.3399 90)
 			(effects
 				(font
@@
 		)
 		(property "Value" "SD05_SOD323"
-			(at 76.2 182.88 90)
+			(at 76.2 182.8799 90)
 			(effects
 				(font
@@
 			(project "BLDC_Motor Controller"
 				(path "/e63e39d7-6ac0-4ffd-8aa3-1841a4541b55/6e5056e0-f286-40ca-8b4a-d506221b7bad"
-					(reference "D2")
+					(reference "D5")
 					(unit 1)
 				)
@@
 		(dnp no)
 		(fields_autoplaced yes)
-		(property "Reference" "D6"
-			(at 106.68 132.3975 90)
+		(property "Reference" "D10"
+			(at 106.68 132.3974 90)
 			(effects
 				(font
@@
 		)
 		(property "Value" "LED_R"
-			(at 106.68 134.9375 90)
+			(at 106.68 134.9374 90)
 			(effects
 				(font
@@
 			(project "BLDC_Motor Controller"
 				(path "/e63e39d7-6ac0-4ffd-8aa3-1841a4541b55/6e5056e0-f286-40ca-8b4a-d506221b7bad"
-					(reference "D6")
+					(reference "D10")
 					(unit 1)
 				)
@@
 		(on_board yes)
 		(dnp no)
-		(property "Reference" "C8"
+		(property "Reference" "C12"
 			(at 88.9 73.66 90)
 			(effects
@@
 			(project "BLDC_Motor Controller"
 				(path "/e63e39d7-6ac0-4ffd-8aa3-1841a4541b55/6e5056e0-f286-40ca-8b4a-d506221b7bad"
-					(reference "C8")
+					(reference "C12")
 					(unit 1)
 				)
@@
 		(on_board yes)
 		(dnp no)
-		(property "Reference" "R3"
+		(property "Reference" "R63"
 			(at 86.36 39.37 0)
 			(effects
@@
 			(project "BLDC_Motor Controller"
 				(path "/e63e39d7-6ac0-4ffd-8aa3-1841a4541b55/6e5056e0-f286-40ca-8b4a-d506221b7bad"
-					(reference "R3")
+					(reference "R63")
 					(unit 1)
 				)
@@
 		(on_board yes)
 		(dnp no)
-		(property "Reference" "C2"
+		(property "Reference" "C8"
 			(at 54.61 26.67 0)
 			(effects
@@
 			(project "BLDC_Motor Controller"
 				(path "/e63e39d7-6ac0-4ffd-8aa3-1841a4541b55/6e5056e0-f286-40ca-8b4a-d506221b7bad"
-					(reference "C2")
+					(reference "C8")
 					(unit 1)
 				)
@@
 		(on_board yes)
 		(dnp no)
-		(property "Reference" "C1"
+		(property "Reference" "C7"
 			(at 29.21 27.94 0)
 			(effects
@@
 			(project "BLDC_Motor Controller"
 				(path "/e63e39d7-6ac0-4ffd-8aa3-1841a4541b55/6e5056e0-f286-40ca-8b4a-d506221b7bad"
-					(reference "C1")
+					(reference "C7")
 					(unit 1)
 				)
@@
 		(on_board yes)
 		(dnp no)
-		(property "Reference" "D4"
+		(property "Reference" "D6"
 			(at 59.3506 166.9575 0)
 			(effects
@@
 			(project "BLDC_Motor Controller"
 				(path "/e63e39d7-6ac0-4ffd-8aa3-1841a4541b55/6e5056e0-f286-40ca-8b4a-d506221b7bad"
-					(reference "D4")
+					(reference "D6")
 					(unit 1)
 				)
@@
 		(on_board yes)
 		(dnp no)
-		(property "Reference" "C10"
+		(property "Reference" "C16"
 			(at 114.3 63.5 0)
 			(effects
@@
 			(project "BLDC_Motor Controller"
 				(path "/e63e39d7-6ac0-4ffd-8aa3-1841a4541b55/6e5056e0-f286-40ca-8b4a-d506221b7bad"
-					(reference "C10")
+					(reference "C16")
 					(unit 1)
 				)
@@
 		(on_board yes)
 		(dnp no)
-		(property "Reference" "J1"
+		(property "Reference" "J2"
 			(at 21.59 167.64 0)
 			(effects
@@
 			(project "BLDC_Motor Controller"
 				(path "/e63e39d7-6ac0-4ffd-8aa3-1841a4541b55/6e5056e0-f286-40ca-8b4a-d506221b7bad"
-					(reference "J1")
+					(reference "J2")
 					(unit 1)
 				)
@@
 		(on_board yes)
 		(dnp no)
-		(property "Reference" "C14"
+		(property "Reference" "C19"
 			(at 180.34 29.21 0)
 			(effects
@@
 			(project "BLDC_Motor Controller"
 				(path "/e63e39d7-6ac0-4ffd-8aa3-1841a4541b55/6e5056e0-f286-40ca-8b4a-d506221b7bad"
-					(reference "C14")
+					(reference "C19")
 					(unit 1)
 				)
@@
 		(on_board yes)
 		(dnp no)
-		(property "Reference" "J2"
+		(property "Reference" "J3"
 			(at 267.97 92.71 0)
 			(effects
@@
 			(project "BLDC_Motor Controller"
 				(path "/e63e39d7-6ac0-4ffd-8aa3-1841a4541b55/6e5056e0-f286-40ca-8b4a-d506221b7bad"
-					(reference "J2")
+					(reference "J3")
 					(unit 1)
 				)
@@
 		(dnp no)
 		(fields_autoplaced yes)
-		(property "Reference" "D5"
-			(at 93.98 132.3975 90)
+		(property "Reference" "D9"
+			(at 93.98 132.3974 90)
 			(effects
 				(font
@@
 		)
 		(property "Value" "LED_G"
-			(at 93.98 134.9375 90)
+			(at 93.98 134.9374 90)
 			(effects
 				(font
@@
 			(project "BLDC_Motor Controller"
 				(path "/e63e39d7-6ac0-4ffd-8aa3-1841a4541b55/6e5056e0-f286-40ca-8b4a-d506221b7bad"
-					(reference "D5")
+					(reference "D9")
 					(unit 1)
 				)
@@
 		(on_board yes)
 		(dnp no)
-		(property "Reference" "C16"
+		(property "Reference" "C21"
 			(at 250.19 125.73 90)
 			(effects
@@
 			(project "BLDC_Motor Controller"
 				(path "/e63e39d7-6ac0-4ffd-8aa3-1841a4541b55/6e5056e0-f286-40ca-8b4a-d506221b7bad"
-					(reference "C16")
+					(reference "C21")
 					(unit 1)
 				)
@@
 		(on_board yes)
 		(dnp no)
-		(property "Reference" "C15"
+		(property "Reference" "C20"
 			(at 195.58 29.21 0)
 			(effects
@@
 			(project "BLDC_Motor Controller"
 				(path "/e63e39d7-6ac0-4ffd-8aa3-1841a4541b55/6e5056e0-f286-40ca-8b4a-d506221b7bad"
-					(reference "C15")
+					(reference "C20")
 					(unit 1)
 				)
@@
 		(dnp no)
 		(fields_autoplaced yes)
-		(property "Reference" "R4"
-			(at 105.41 119.38 0)
+		(property "Reference" "R8"
+			(at 105.41 119.3799 0)
 			(effects
 				(font
@@
 		)
 		(property "Value" "1k"
-			(at 105.41 121.92 0)
+			(at 105.41 121.9199 0)
 			(effects
 				(font
@@
 			(project "BLDC_Motor Controller"
 				(path "/e63e39d7-6ac0-4ffd-8aa3-1841a4541b55/6e5056e0-f286-40ca-8b4a-d506221b7bad"
-					(reference "R4")
+					(reference "R8")
 					(unit 1)
 				)
@@
 		(on_board yes)
 		(dnp no)
-		(property "Reference" "J3"
+		(property "Reference" "J4"
 			(at 270.51 125.73 0)
 			(effects
@@
 			(project "BLDC_Motor Controller"
 				(path "/e63e39d7-6ac0-4ffd-8aa3-1841a4541b55/6e5056e0-f286-40ca-8b4a-d506221b7bad"
-					(reference "J3")
+					(reference "J4")
 					(unit 1)
 				)
@@
 		(on_board yes)
 		(dnp no)
-		(property "Reference" "D15"
+		(property "Reference" "D11"
 			(at 247.3406 90.7322 0)
 			(effects
@@
 			(project "BLDC_Motor Controller"
 				(path "/e63e39d7-6ac0-4ffd-8aa3-1841a4541b55/6e5056e0-f286-40ca-8b4a-d506221b7bad"
-					(reference "D15")
+					(reference "D11")
 					(unit 1)
 				)
@@
 		(on_board yes)
 		(dnp no)
-		(property "Reference" "C3"
+		(property "Reference" "C9"
 			(at 60.96 26.67 0)
 			(effects
@@
 			(project "BLDC_Motor Controller"
 				(path "/e63e39d7-6ac0-4ffd-8aa3-1841a4541b55/6e5056e0-f286-40ca-8b4a-d506221b7bad"
-					(reference "C3")
+					(reference "C9")
 					(unit 1)
 				)
@@
 		(dnp no)
 		(fields_autoplaced yes)
-		(property "Reference" "U1"
+		(property "Reference" "U2"
 			(at 163.4841 139.7 0)
 			(effects
@@
 			(project "BLDC_Motor Controller"
 				(path "/e63e39d7-6ac0-4ffd-8aa3-1841a4541b55/6e5056e0-f286-40ca-8b4a-d506221b7bad"
-					(reference "U1")
+					(reference "U2")
 					(unit 1)
 				)
@@
 		(on_board yes)
 		(dnp no)
-		(property "Reference" "C4"
+		(property "Reference" "C10"
 			(at 67.31 26.67 0)
 			(effects
@@
 			(project "BLDC_Motor Controller"
 				(path "/e63e39d7-6ac0-4ffd-8aa3-1841a4541b55/6e5056e0-f286-40ca-8b4a-d506221b7bad"
-					(reference "C4")
+					(reference "C10")
 					(unit 1)
 				)
@@
 		(on_board yes)
 		(dnp no)
-		(property "Reference" "D3"
+		(property "Reference" "D8"
 			(at 82.55 166.37 0)
 			(effects
@@
 			(project "BLDC_Motor Controller"
 				(path "/e63e39d7-6ac0-4ffd-8aa3-1841a4541b55/6e5056e0-f286-40ca-8b4a-d506221b7bad"
-					(reference "D3")
+					(reference "D8")
 					(unit 1)
 				)
@@
 		(dnp no)
 		(fields_autoplaced yes)
-		(property "Reference" "R2"
-			(at 92.71 119.38 0)
+		(property "Reference" "R7"
+			(at 92.71 119.3799 0)
 			(effects
 				(font
@@
 		)
 		(property "Value" "1k"
-			(at 92.71 121.92 0)
+			(at 92.71 121.9199 0)
 			(effects
 				(font
@@
 			(project "BLDC_Motor Controller"
 				(path "/e63e39d7-6ac0-4ffd-8aa3-1841a4541b55/6e5056e0-f286-40ca-8b4a-d506221b7bad"
-					(reference "R2")
+					(reference "R7")
 					(unit 1)
 				)
@@
 		(on_board yes)
 		(dnp no)
-		(property "Reference" "C5"
+		(property "Reference" "C11"
 			(at 73.66 26.67 0)
 			(effects
@@
 			(project "BLDC_Motor Controller"
 				(path "/e63e39d7-6ac0-4ffd-8aa3-1841a4541b55/6e5056e0-f286-40ca-8b4a-d506221b7bad"
-					(reference "C5")
+					(reference "C11")
 					(unit 1)
 				)
@@
 		(on_board yes)
 		(dnp no)
-		(property "Reference" "C13"
+		(property "Reference" "C18"
 			(at 132.08 64.77 0)
 			(effects
@@
 			(project "BLDC_Motor Controller"
 				(path "/e63e39d7-6ac0-4ffd-8aa3-1841a4541b55/6e5056e0-f286-40ca-8b4a-d506221b7bad"
-					(reference "C13")
+					(reference "C18")
 					(unit 1)
 				)
@@
 		(on_board yes)
 		(dnp no)
-		(property "Reference" "C7"
+		(property "Reference" "C14"
 			(at 86.36 26.67 0)
 			(effects
@@
 			(project "BLDC_Motor Controller"
 				(path "/e63e39d7-6ac0-4ffd-8aa3-1841a4541b55/6e5056e0-f286-40ca-8b4a-d506221b7bad"
-					(reference "C7")
+					(reference "C14")
 					(unit 1)
 				)
@@
 		(on_board yes)
 		(dnp no)
-		(property "Reference" "C9"
+		(property "Reference" "C13"
 			(at 90.17 101.6 90)
 			(effects
@@
 			(project "BLDC_Motor Controller"
 				(path "/e63e39d7-6ac0-4ffd-8aa3-1841a4541b55/6e5056e0-f286-40ca-8b4a-d506221b7bad"
-					(reference "C9")
+					(reference "C13")
 					(unit 1)
 				)
@@
 		(on_board yes)
 		(dnp no)
-		(property "Reference" "C11"
+		(property "Reference" "C17"
 			(at 125.73 36.83 0)
 			(effects
@@
 			(project "BLDC_Motor Controller"
 				(path "/e63e39d7-6ac0-4ffd-8aa3-1841a4541b55/6e5056e0-f286-40ca-8b4a-d506221b7bad"
-					(reference "C11")
+					(reference "C17")
 					(unit 1)
 				)
