File: Projects/Fresu/BLDC Motor Controller/Design/rev01/rev01_1/BLDC_Motor Controller/BLDC_Motor Controller.kicad_pcb (KiCad board)
At the start: 4 copper layers, 100 x 75 mm, 179 parts, among them CN1 XT60PW-M, J1 Conn_01x08, J2 Conn_01x06, J3 Conn_01x03, J4 7461084, J5 7461084, J6 7461084, J7 Conn_01x06, J8 XH-2PWBPZ, J9 TYPE-C-31-M-12, Q1 HSBA15810C, Q2 HSBA15810C, Q3 HSBA15810C, Q4 HSBA15810C, Q5 HSBA15810C, Q6 HSBA15810C, SW1 PTS526SK15SMTR2LFS, U1 STM32F405RGTx, U2 DRV8302_DCA_56, U3 S4B-XH-SM4-TB-(LF)(SN), U4 SN65HVD230, U5 AMS1117-3.3, U6 PUSB3AB6Z, Y1 8MHz

Commit message: Update 20
First layout completed, all tracks laid
Parts:
- removed C6: 100nF, Capacitor_SMD:C_0603_1608Metric
- D10: moved to F.Cu
- R16, R17, R20, R21, R22, R23, R57: moved to B.Cu
- moved C56 257.6 mm to (237.9, 120.0), turned to 180 degrees
- moved R57 85.7 mm to (183.2, 140.8), turned to 180 degrees
- moved C1 43.5 mm to (198.8, 130.7)
- moved R56 41.7 mm to (228.5, 112.6), turned to 180 degrees
- moved R17 28.4 mm to (191.3, 144.8), turned to -90 degrees
- moved R23 28.0 mm to (194.3, 140.6), turned to -90 degrees
- moved R21 25.8 mm to (194.1, 143.4), turned to -45 degrees
- moved R22 12.1 mm to (211.7, 147.2), turned to 0 degrees
- moved R16 10.3 mm to (211.8, 150.4), turned to 0 degrees
- moved R20 8.73 mm to (211.8, 148.7), turned to 0 degrees
- moved R53 7.76 mm to (165.4, 164.1), turned to -90 degrees
- moved C58 6.41 mm to (183.3, 139.7), turned to 180 degrees
- moved D14 5.09 mm to (222.1, 114.9), turned to -90 degrees
- moved D2 3.56 mm to (173.1, 135.0), turned to 90 degrees
- moved C22 3.55 mm to (212.0, 136.3)
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Connections:
- net CAN_RX renamed CAN-
- net CAN_TX renamed CAN+
- net Net-(D13-A) renamed /STEP-DOWN/+3v3Vout
Routing:
- net +5V: track 0.00 -> 162.6 mm, vias 0 -> 8
- net +3V3: track 14.9 -> 175.1 mm, vias 0 -> 12
- net GND: track 27.5 -> 149.0 mm, vias 103 -> 245
- net AN_IN: track 1.78 -> 80.6 mm, vias 1 -> 2
- net +VDC: track 0.00 -> 64.5 mm, vias 120 -> 127
- net /MCU/NRST: track 4.05 -> 46.9 mm, vias 0 -> 4
- net /USB/USB-C_P: track 0.00 -> 37.6 mm, vias 0 -> 2
- net HALL_1_OUT: track 1.98 -> 38.3 mm, vias 1 -> 2
- net /USB/USB-C_N: track 0.00 -> 36.0 mm, vias 0 -> 2
- net HALL_3_OUT: track 1.72 -> 36.8 mm, vias 1 -> 2
- net TEMP_MOTOR: track 1.51 -> 34.6 mm, vias 1 -> 2
- net HALL_2_OUT: track 2.11 -> 32.8 mm, vias 1 -> 2
- net CAN-: track 0.00 -> 28.0 mm
- net SENS1: track 0.00 -> 27.8 mm, vias 0 -> 1
- net SENS3: track 0.00 -> 27.6 mm, vias 0 -> 1
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- added copper zone on F.Cu, net +3V3
- added copper zone on F.Cu, net /STEP-DOWN/+3v3Vout

Commit message: Update 21
Now all tracks are laid, working on DRC
Routing:
- net +3V3: track 175.1 -> 205.2 mm, vias 12 -> 17
- net GND: track 149.0 -> 156.1 mm, vias 245 -> 252
- net Net-(U2-AVDD): track 0.00 -> 3.04 mm
- net Net-(D15-A): track 0.00 -> 1.89 mm
- net SENS3: track 27.6 -> 29.3 mm
- net SENS2: track 27.4 -> 28.5 mm
- net L1: track 13.4 -> 12.5 mm
- net H2: track 14.9 -> 14.2 mm
