File: Projects/Fresu/BLDC Motor Controller/Design/rev01/rev01_1/BLDC_Motor Controller/Block Diagram.kicad_sch (KiCad schematic)
At the start: 0 parts

Commit message: Update 4
Started Block Diagram page
Other:
- note added: "0-60V"
- note added: "BLOCK DIAGRAM"
- note added: "CAN"
- note added: "COM"
- note added: "HALL/ENCODER"
- note added: "MCU"
- note added: "MOSFET"
- note added: "MOSFET DRIVER"
- note added: "MOTOR"
- note added: "SERVO"
- note added: "TEMP_SENSOR"
- note added: "USB"
- note added: "V_SUPPLY"
Changed lines of the file:
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@@
 (kicad_sch (version 20230121) (generator eeschema)
   (paper "A4")
+  (polyline (pts (xy 187.96 134.62) (xy 163.83 134.62))
+    (stroke (width 0) (type default))
+  )
+  (polyline (pts (xy 90.17 95.25) (xy 90.17 106.68))
+    (stroke (width 0) (type default))
+  )
+  (polyline (pts (xy 109.22 137.16) (xy 152.4 137.16))
+    (stroke (width 0) (type default))
+  )
+  (polyline (pts (xy 109.22 130.81) (xy 109.22 142.24))
+    (stroke (width 0) (type default))
+  )
+  (polyline (pts (xy 236.22 99.06) (xy 247.65 99.06))
+    (stroke (width 2) (type solid))
+  )
+  (polyline (pts (xy 236.22 127) (xy 236.22 55.88))
+    (stroke (width 0) (type solid))
+  )
+  (polyline (pts (xy 90.17 142.24) (xy 109.22 142.24))
+    (stroke (width 0) (type default))
+  )
+  (polyline (pts (xy 143.51 118.11) (xy 143.51 77.47))
+    (stroke (width 0) (type default))
+  )
+  (polyline (pts (xy 125.73 60.96) (xy 137.16 60.96))
+    (stroke (width 2) (type default))
+  )
+  (polyline (pts (xy 170.18 143.51) (xy 170.18 154.94))
+    (stroke (width 0) (type default))
+  )
+  (polyline (pts (xy 152.4 80.01) (xy 152.4 137.16))
+    (stroke (width 0) (type default))
+  )
+  (polyline (pts (xy 247.65 92.71) (xy 267.97 92.71))
+    (stroke (width 0) (type default))
+  )
+  (polyline (pts (xy 191.77 93.98) (xy 222.25 93.98))
+    (stroke (width 0) (type default))
+  )
+  (polyline (pts (xy 163.83 80.01) (xy 163.83 134.62))
+    (stroke (width 0) (type default))
+  )
+  (polyline (pts (xy 125.73 55.88) (xy 125.73 67.31))
+    (stroke (width 0) (type default))
+  )
+  (polyline (pts (xy 267.97 92.71) (xy 267.97 104.14))
+    (stroke (width 0) (type default))
+  )
+  (polyline (pts (xy 187.96 143.51) (xy 187.96 134.62))
+    (stroke (width 0) (type default))
+  )
+  (polyline (pts (xy 191.77 82.55) (xy 191.77 93.98))
+    (stroke (width 0) (type default))
+  )
+  (polyline (pts (xy 247.65 104.14) (xy 267.97 104.14))
+    (stroke (width 0) (type default))
+  )
+  (polyline (pts (xy 176.53 143.51) (xy 176.53 154.94))
+    (stroke (width 0) (type default))
+  )
+  (polyline (pts (xy 157.48 80.01) (xy 157.48 143.51))
+    (stroke (width 0) (type default))
+  )
+  (polyline (pts (xy 185.42 74.93) (xy 228.6 74.93))
+    (stroke (width 0) (type default))
+  )
+  (polyline (pts (xy 95.25 67.31) (xy 125.73 67.31))
+    (stroke (width 0) (type default))
+  )
+  (polyline (pts (xy 95.25 55.88) (xy 125.73 55.88))
+    (stroke (width 0) (type default))
+  )
+  (polyline (pts (xy 129.54 111.76) (xy 129.54 123.19))
+    (stroke (width 0) (type default))
+  )
+  (polyline (pts (xy 111.76 101.6) (xy 134.62 101.6))
+    (stroke (width 0) (type default))
+  )
+  (polyline (pts (xy 137.16 55.88) (xy 137.16 62.23))
+    (stroke (width 0) (type solid))
+  )
+  (polyline (pts (xy 236.22 55.88) (xy 137.16 55.88))
+    (stroke (width 0) (type solid))
+  )
+  (polyline (pts (xy 90.17 111.76) (xy 90.17 123.19))
+    (stroke (width 0) (type default))
+  )
+  (polyline (pts (xy 222.25 82.55) (xy 222.25 93.98))
+    (stroke (width 0) (type default))
+  )
+  (polyline (pts (xy 90.17 106.68) (xy 111.76 106.68))
+    (stroke (width 0) (type default))
+  )
+  (polyline (pts (xy 90.17 130.81) (xy 109.22 130.81))
+    (stroke (width 0) (type default))
+  )
+  (polyline (pts (xy 129.54 68.58) (xy 149.86 68.58))
+    (stroke (width 0) (type default))
+  )
+  (polyline (pts (xy 90.17 90.17) (xy 111.76 90.17))
+    (stroke (width 0) (type default))
+  )
+  (polyline (pts (xy 228.6 63.5) (xy 228.6 74.93))
+    (stroke (width 0) (type default))
+  )
+  (polyline (pts (xy 134.62 101.6) (xy 134.62 73.66))
+    (stroke (width 0) (type default))
+  )
+  (polyline (pts (xy 134.62 143.51) (xy 134.62 154.94))
+    (stroke (width 0) (type default))
+  )
+  (polyline (pts (xy 111.76 78.74) (xy 111.76 90.17))
+    (stroke (width 0) (type default))
+  )
+  (polyline (pts (xy 90.17 78.74) (xy 111.76 78.74))
+    (stroke (width 0) (type default))
+  )
+  (polyline (pts (xy 200.66 143.51) (xy 200.66 154.94))
+    (stroke (width 0) (type default))
+  )
+  (polyline (pts (xy 191.77 82.55) (xy 222.25 82.55))
+    (stroke (width 0) (type default))
+  )
+  (polyline (pts (xy 90.17 78.74) (xy 90.17 90.17))
+    (stroke (width 0) (type default))
+  )
+  (polyline (pts (xy 111.76 83.82) (xy 129.54 83.82))
+    (stroke (width 0) (type default))
+  )
+  (polyline (pts (xy 168.91 62.23) (xy 168.91 80.01))
+    (stroke (width 0) (type default))
+  )
+  (polyline (pts (xy 137.16 62.23) (xy 137.16 127))
+    (stroke (width 0) (type solid))
+  )
+  (polyline (pts (xy 90.17 111.76) (xy 129.54 111.76))
+    (stroke (width 0) (type default))
+  )
+  (polyline (pts (xy 90.17 130.81) (xy 90.17 142.24))
+    (stroke (width 0) (type default))
+  )
+  (polyline (pts (xy 90.17 123.19) (xy 129.54 123.19))
+    (stroke (width 0) (type default))
+  )
+  (polyline (pts (xy 134.62 143.51) (xy 170.18 143.51))
+    (stroke (width 0) (type default))
+  )
+  (polyline (pts (xy 134.62 154.94) (xy 170.18 154.94))
+    (stroke (width 0) (type default))
+  )
+  (polyline (pts (xy 137.16 127) (xy 236.22 127))
+    (stroke (width 0) (type solid))
+  )
+  (polyline (pts (xy 185.42 63.5) (xy 228.6 63.5))
+    (stroke (width 0) (type default))
+  )
+  (polyline (pts (xy 143.51 77.47) (xy 149.86 77.47))
+    (stroke (width 0) (type default))
+  )
+  (polyline (pts (xy 134.62 73.66) (xy 149.86 73.66))
+    (stroke (width 0) (type default))
+  )
+  (polyline (pts (xy 149.86 62.23) (xy 168.91 62.23))
+    (stroke (width 0) (type default))
+  )
+  (polyline (pts (xy 90.17 95.25) (xy 111.76 95.25))
+    (stroke (width 0) (type default))
+  )
+  (polyline (pts (xy 111.76 95.25) (xy 111.76 106.68))
+    (stroke (width 0) (type default))
+  )
+  (polyline (pts (xy 185.42 63.5) (xy 185.42 74.93))
+    (stroke (width 0) (type default))
+  )
+  (polyline (pts (xy 149.86 62.23) (xy 149.86 80.01))
+    (stroke (width 0) (type default))
+  )
+  (polyline (pts (xy 129.54 83.82) (xy 129.54 68.58))
+    (stroke (width 0) (type default))
+  )
+  (polyline (pts (xy 176.53 154.94) (xy 200.66 154.94))
+    (stroke (width 0) (type default))
+  )
+  (polyline (pts (xy 149.86 80.01) (xy 168.91 80.01))
+    (stroke (width 0) (type default))
+  )
+  (polyline (pts (xy 247.65 92.71) (xy 247.65 104.14))
+    (stroke (width 0) (type default))
+  )
+  (polyline (pts (xy 176.53 143.51) (xy 200.66 143.51))
+    (stroke (width 0) (type default))
+  )
+  (polyline (pts (xy 129.54 118.11) (xy 143.51 118.11))
+    (stroke (width 0) (type default))
+  )
+  (polyline (pts (xy 95.25 55.88) (xy 95.25 67.31))
+    (stroke (width 0) (type default))
+  )
+  (text "MCU" (at 153.67 73.66 0)
+    (effects (font (size 3 3) bold) (justify left bottom))
+  )
+  (text "MOSFET" (at 195.58 90.17 0)
+    (effects (font (size 3 3) bold) (justify left bottom))
+  )
+  (text "V_SUPPLY" (at 99.06 63.5 0)
+    (effects (font (size 3 3) bold) (justify left bottom))
+  )
+  (text "MOTOR" (at 248.92 100.33 0)
+    (effects (font (size 3 3) bold) (justify left bottom))
+  )
+  (text "TEMP_SENSOR" (at 135.89 151.13 0)
+    (effects (font (size 3 3) bold) (justify left bottom))
+  )
+  (text "BLOCK DIAGRAM" (at 124.46 30.48 0)
+    (effects (font (size 5 5) (thickness 1) bold) (justify left bottom))
+  )
+  (text "USB\n" (at 95.25 86.36 0)
+    (effects (font (size 3 3) bold) (justify left bottom))
+  )
+  (text "HALL/ENCODER\n	" (at 91.44 124.46 0)
+    (effects (font (size 3 3) bold) (justify left bottom))
+  )
+  (text "SERVO" (at 180.34 151.13 0)
+    (effects (font (size 3 3) bold) (justify left bottom))
+  )
+  (text "COM\n" (at 93.98 138.43 0)
+    (effects (font (size 3 3) bold) (justify left bottom))
+  )
+  (text "0-60V" (at 107.95 55.88 0)
+    (effects (font (size 2 2) bold) (justify left bottom))
+  )
+  (text "MOSFET DRIVER\n" (at 189.23 71.12 0)
+    (effects (font (size 3 3) bold) (justify left bottom))
+  )
+  (text "CAN\n\n" (at 95.25 107.95 0)
+    (effects (font (size 3 3) bold) (justify left bottom))
+  )
 )
