File: Projects/Fresu/BLDC Motor Controller/Design/rev01/rev01_1/BLDC_Motor Controller/MOSFETS.kicad_sch (KiCad schematic)
At the start: 0 parts

Commit message: UPDATE 6
Completed MCU schematic Page
Parts:
- added C18, C26: 10n, symbol Device:C
- added C19: 120p, symbol Device:C
- added C20, C21, C22, C23, C25: 2u2, symbol Device:C
- added C24: 22n, symbol Device:C
- added C27, C28, C29, C30, C31, C32, C33, C34, C35: 10u, symbol Device:C
- added C36, C37, C38, C39, C40, C41: 100n, symbol Device:C
- added D7: PMEG6020ELR, Diode_SMD:Nexperia_CFP3_SOD-123W, symbol Diode:PMEG6020ELR
- added D8: BAT60A, Diode_SMD:D_SOD-323, symbol Diode:BAT60A
- added L1: 22u, symbol Device:L
- added NT1: NetTie_2, symbol Device:NetTie_2
- added R11: 16k, symbol Device:R
- added R12: 205K, symbol Device:R
- added R13: 10k, symbol Device:R
- added R14: 1M, symbol Device:R
- added R15, R17, R19, R21: 18K, symbol Device:R
- added R16: 3K3, symbol Device:R
- added R18, R20, R22: 2K2, symbol Device:R
- added U2: DRV8302_DCA_56, DCA56_6P35X3P61, symbol DRV8302:DRV8302_DCA_56
Connections:
- new net: C25.2, U2.27 (AVDD)
- new net: C18.2, R11.1
- new net: C18.1, C19.1
- new net +3V3: U2.24 (REF), U2.9 (M_OC)
- new net +5V: D8.1 (K)
- new net +5V_DRV: C27.2, C28.2, C29.2, D8.2 (A), L1.2, R15.2
- new net +VDC: C30.2, C31.2, C32.2, C33.2, C34.2, C35.2, C39.2, C40.2, C41.2, U2.29 (PVDD1), U2.53 (PVDD2), U2.54 (PVDD2)
- new net BIAS: R14.1, U2.49 (BIAS)
- new net BR_S01: U2.25 (SO1)
- new net BR_S02: U2.26 (SO2)
- new net BST_A: C36.2, U2.48 (BST_A)
- new net BST_B: C37.2, U2.43 (BST_B)
- new net BST_BK: C26.1, U2.52 (BST_BK)
- new net BST_C: C38.2, U2.38 (BST_C)
- new net COMP: C19.2, R11.2, U2.2 (COMP)
- new net CP1: C24.2, U2.14 (CP1)
- new net CP2: C24.1, U2.15 (CP2)
- new net DC_CAL: U2.12 (DC_CAL)
- new net DTC: R13.2, U2.7 (DTC)
- new net DVDD: NT1.1, U2.23 (DVDD)
- new net EN_GATE: U2.16 (EN_GATE)
- new net FAULT: U2.6 (*FAULT)
- new net GND: C20.1, C21.1, C22.1, C23.1, C25.1, C27.1, C28.1, C29.1, C30.1, C31.1, C32.1, C33.1, C34.1, C35.1, C39.1, C40.1, C41.1, D7.2 (A), R12.1, R13.1, R14.2, R16.1, R18.1, R20.1, R22.1, U2.10 (GAIN), U2.28 (AGND), U2.57 (EPAD), U2.8 (M_PWM)
- new net GVDD: C22.2, C23.2, U2.13 (GVDD)
- new net H1: U2.17 (INH_A)
- new net H1_LOW: U2.44 (SL_A)
- new net H1_VS: C36.1, R21.2, U2.46 (SH_A)
- new net H2: U2.19 (INH_B)
- new net H2_LOW: U2.39 (SL_B)
- new net H2_VS: C37.1, R19.2, U2.41 (SH_B)
- new net H3: U2.21 (INH_C)
- new net H3_LOW: U2.34 (SL_C)
- new net H3_VS: C38.1, R17.2, U2.36 (SH_C)
- new net L1: U2.18 (INL_A)
- new net L2: U2.20 (INL_B)
- new net L3: U2.22 (INL_C)
- new net M_H1: U2.47 (GH_A)
- new net M_H2: U2.42 (GH_B)
- new net M_H3: U2.37 (GH_C)
- new net M_L1: U2.45 (GL_A)
- new net M_L2: U2.40 (GL_B)
- new net M_L3: U2.35 (GL_C)
- new net OC_ADJ: C20.2, C21.2, NT1.2, U2.11 (OC_ADJ)
- new net PH: C26.2, D7.1 (K), L1.1, U2.50 (PH), U2.51 (PH)
- new net RT_CLK: R12.2, U2.1 (RT_CLK)
- new net S1_N: U2.33 (SN1)
- new net S1_P: U2.32 (SP1)
- new net S2_N: U2.31 (SN2)
- new net S2_P: U2.30 (SP2)
- new net SENS1: R17.1, R18.2
- new net SENS2: R19.1, R20.2
- new net SENS3: R21.1, R22.2
- new net VSENSE: U2.3 (VSENSE)
- new net V_SENSE: R15.1, R16.2
- no-connect marks 0 -> 4
Other:
- note added: "ADD FAULT PULL UP"
- note added: "BOOTSTRAP CAPs"
- note added: "Hx_VS"
- note added: "INPUT PORTS"
- note added: "MCU SENSING FEEDBACK FOR EACH PHASE"
- note added: "OUTPUT PORTS"
- note added: "PHASE_1"
- note added: "PHASE_2"
- note added: "PHASE_3"
- note added: "SENSE 1 - PHASE 1"
- note added: "SENSE 2 - PHASE 2"

Commit message: UPDATE 7
COMPLETED MOSFET SCHEMATIC
Parts:
- removed C18, C26: 10n, symbol Device:C
- removed C19: 120p, symbol Device:C
- removed C20, C21, C22, C23, C25: 2u2, symbol Device:C
- removed C24: 22n, symbol Device:C
- removed C27, C28, C29, C30, C31, C32, C33, C34, C35: 10u, symbol Device:C
- removed C36, C37, C38, C39, C40, C41: 100n, symbol Device:C
- removed D7: PMEG6020ELR, Diode_SMD:Nexperia_CFP3_SOD-123W, symbol Diode:PMEG6020ELR
- removed D8: BAT60A, Diode_SMD:D_SOD-323, symbol Diode:BAT60A
- removed L1: 22u, symbol Device:L
- removed NT1: NetTie_2, symbol Device:NetTie_2
- removed R11: 16k, symbol Device:R
- removed R12: 205K, symbol Device:R
- removed R13: 10k, symbol Device:R
- removed R14: 1M, symbol Device:R
- removed R15, R17, R19, R21: 18K, symbol Device:R
- removed R16: 3K3, symbol Device:R
- removed R18, R20, R22: 2K2, symbol Device:R
- removed U2: DRV8302_DCA_56, DCA56_6P35X3P61, symbol DRV8302:DRV8302_DCA_56
- added C42, C43: 2N2, symbol Device:C
- added J4, J5, J6: 7461084, symbol Connector_Generic:Conn_01x01
- added NT2, NT3, NT4, NT5, NT6, NT7: NetTie_2, symbol Device:NetTie_2
- added Q1, Q2, Q3, Q4, Q5, Q6: HSBA15810C, symbol Simulation_SPICE:NMOS
- added R23, R24, R26, R27, R32, R33: 4R7, symbol Device:R
- added R25, R28, R36: 39K, symbol Device:R
- added R29, R37: 0R001, symbol Device:R_Shunt
- added R30, R31, R34, R35: 100R, symbol Device:R
Connections:
- net +VDC: now also Q1.1 (D), Q3.1 (D), Q5.1 (D)
- net GND: now also NT3.1, R25.1, R28.1, R29.4, R36.1, R37.4
- net H1_LOW: now also NT7.2, Q6.3 (S)
- net H1_VS: now also NT6.1
- net H2_LOW: now also NT5.2, Q4.3 (S)
- net H2_VS: now also NT4.1
- net H3_LOW: now also NT3.2, Q2.3 (S)
- net H3_VS: now also NT2.1
- net M_H1: now also R32.1
- net M_H2: now also R26.1
- net M_H3: now also R23.1
- net M_L1: now also R33.1
- net M_L2: now also R27.1
- net M_L3: now also R24.1
- net S1_N: now also C43.1, R34.1
- net S1_P: now also C43.2, R35.1
- net S2_N: now also C42.1, R30.1
- net S2_P: now also C42.2, R31.1
- new net: NT7.1, R37.1
- new net: NT5.1, R29.1
- new net M_H1_RG: Q5.2 (G), R32.2
- new net M_H2_RG: Q3.2 (G), R26.2
- new net M_H3_RG: Q1.2 (G), R23.2
- new net M_L1_RG: Q6.2 (G), R33.2, R36.2
- new net M_L2_RG: Q4.2 (G), R27.2, R28.2
- new net M_L3_RG: Q2.2 (G), R24.2, R25.2
- new net PHASE_1: J4.1 (Pin_1), NT6.2, Q5.3 (S), Q6.1 (D)
- new net PHASE_2: J5.1 (Pin_1), NT4.2, Q3.3 (S), Q4.1 (D)
- new net PHASE_3: J6.1 (Pin_1), NT2.2, Q1.3 (S), Q2.1 (D)
- new net SH1_N: R34.2, R37.2
- new net SH1_P: R35.2, R37.3
- new net SH2_N: R29.2, R30.2
- new net SH2_P: R29.3, R31.2
- no-connect marks 4 -> 0
Other:
- note added: "MCU SENSING FEEDBACK FOR EAC PHASE"
- note added: "OUTPUT PHASE 1"
- note added: "OUTPUT PHASE 2"
- note added: "OUTPUT PHASE 3"
- note added: "PHASE 1"
- note added: "PHASE 2"
- note added: "PHASE 3"
- note added: "Q_CONTROL"
- note added: "Q_SOURCES"
- note added: "SENSE 1"
- note added: "SENSE 2"
- note removed: "ADD FAULT PULL UP"
- note removed: "BOOTSTRAP CAPs"
- note removed: "INPUT PORTS"
- note removed: "MCU SENSING FEEDBACK FOR EACH PHASE"
- note removed: "OUTPUT PORTS"
- note removed: "PHASE_1"
- note removed: "PHASE_2"
- note removed: "PHASE_3"
- note removed: "SENSE 1 - PHASE 1"
- note removed: "SENSE 2 - PHASE 2"

Commit message: Update 13
Added:
1) USB Schematic
2) footprints to all parts
Parts:
- C42, C43: footprint (none) -> Capacitor_SMD:C_0603_1608Metric
- J4, J5, J6: footprint (none) -> 7461084:WE_7461084
- NT2, NT4, NT6: footprint (none) -> NetTie:NetTie-2_SMD_Pad0.5mm
- NT3, NT5, NT7: footprint (none) -> DF_ESC_Footprint_Library:NetTie_SMD_Pad_3.00mm
- Q1, Q2, Q3, Q4, Q5, Q6: footprint (none) -> Package_DFN_QFN:PQFN-8-EP_6x5mm_P1.27mm_Generic
- R23, R24, R25, R26, R27, R28, R30, R31, R32, R33, R34, R35, R36: footprint (none) -> Resistor_SMD:R_0603_1608Metric_Pad0.98x0.95mm_HandSolder
- R29, R37: footprint (none) -> DF_ESC_Footprint_Library:RES-SMD_L7.0-W6.7
Changed lines of the file:
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@@
       (effects (font (size 1.27 1.27)) (justify right))
     )
-    (property "Footprint" "" (at 213.36 114.3 0)
+    (property "Footprint" "DF_ESC_Footprint_Library:NetTie_SMD_Pad_3.00mm" (at 213.36 114.3 0)
       (effects (font (size 1.27 1.27)) hide)
     )
@@
       (effects (font (size 1.27 1.27)))
     )
-    (property "Footprint" "" (at 127 64.008 90)
+    (property "Footprint" "Resistor_SMD:R_0603_1608Metric_Pad0.98x0.95mm_HandSolder" (at 127 64.008 90)
       (effects (font (size 1.27 1.27)) hide)
     )
@@
       (effects (font (size 1.27 1.27)))
     )
-    (property "Footprint" "" (at 191.77 100.838 90)
+    (property "Footprint" "Resistor_SMD:R_0603_1608Metric_Pad0.98x0.95mm_HandSolder" (at 191.77 100.838 90)
       (effects (font (size 1.27 1.27)) hide)
     )
@@
       (effects (font (size 1.27 1.27)) (justify right))
     )
-    (property "Footprint" "" (at 82.55 102.87 0)
+    (property "Footprint" "DF_ESC_Footprint_Library:NetTie_SMD_Pad_3.00mm" (at 82.55 102.87 0)
       (effects (font (size 1.27 1.27)) hide)
     )
@@
       (effects (font (size 1.27 1.27)))
     )
-    (property "Footprint" "" (at 66.04 118.618 90)
+    (property "Footprint" "Resistor_SMD:R_0603_1608Metric_Pad0.98x0.95mm_HandSolder" (at 66.04 118.618 90)
       (effects (font (size 1.27 1.27)) hide)
     )
@@
       (effects (font (size 1.27 1.27)))
     )
-    (property "Footprint" "" (at 132.08 118.618 90)
+    (property "Footprint" "Resistor_SMD:R_0603_1608Metric_Pad0.98x0.95mm_HandSolder" (at 132.08 118.618 90)
       (effects (font (size 1.27 1.27)) hide)
     )
@@
       (effects (font (size 1.27 1.27)))
     )
-    (property "Footprint" "" (at 134.62 74.93 0)
+    (property "Footprint" "NetTie:NetTie-2_SMD_Pad0.5mm" (at 134.62 74.93 0)
       (effects (font (size 1.27 1.27)) hide)
     )
@@
       (effects (font (size 1.27 1.27)))
     )
-    (property "Footprint" "" (at 60.96 64.008 90)
+    (property "Footprint" "Resistor_SMD:R_0603_1608Metric_Pad0.98x0.95mm_HandSolder" (at 60.96 64.008 90)
       (effects (font (size 1.27 1.27)) hide)
     )
@@
       (effects (font (size 1.27 1.27)) (justify right))
     )
-    (property "Footprint" "" (at 70.358 95.25 90)
+    (property "Footprint" "Resistor_SMD:R_0603_1608Metric_Pad0.98x0.95mm_HandSolder" (at 70.358 95.25 90)
       (effects (font (size 1.27 1.27)) hide)
     )
@@
       (effects (font (size 1.27 1.27)) (justify left))
     )
-    (property "Footprint" "" (at 85.09 59.69 0)
+    (property "Footprint" "Package_DFN_QFN:PQFN-8-EP_6x5mm_P1.27mm_Generic" (at 85.09 59.69 0)
       (effects (font (size 1.27 1.27)) hide)
     )
@@
       (effects (font (size 1.27 1.27)))
     )
-    (property "Footprint" "" (at 66.04 122.682 90)
+    (property "Footprint" "Resistor_SMD:R_0603_1608Metric_Pad0.98x0.95mm_HandSolder" (at 66.04 122.682 90)
       (effects (font (size 1.27 1.27)) hide)
     )
@@
       (effects (font (size 1.27 1.27)) (justify right))
     )
-    (property "Footprint" "" (at 201.168 106.68 90)
+    (property "Footprint" "Resistor_SMD:R_0603_1608Metric_Pad0.98x0.95mm_HandSolder" (at 201.168 106.68 90)
       (effects (font (size 1.27 1.27)) hide)
     )
@@
       (effects (font (size 1.27 1.27)) (justify left))
     )
-    (property "Footprint" "" (at 215.9 96.52 0)
+    (property "Footprint" "Package_DFN_QFN:PQFN-8-EP_6x5mm_P1.27mm_Generic" (at 215.9 96.52 0)
       (effects (font (size 1.27 1.27)) hide)
     )
@@
       (effects (font (size 1.27 1.27)))
     )
-    (property "Footprint" "" (at 68.58 74.93 0)
+    (property "Footprint" "NetTie:NetTie-2_SMD_Pad0.5mm" (at 68.58 74.93 0)
       (effects (font (size 1.27 1.27)) hide)
     )
@@
       (effects (font (size 1.27 1.27)))
     )
-    (property "Footprint" "" (at 132.08 122.682 90)
+    (property "Footprint" "Resistor_SMD:R_0603_1608Metric_Pad0.98x0.95mm_HandSolder" (at 132.08 122.682 90)
       (effects (font (size 1.27 1.27)) hide)
     )
@@
       (effects (font (size 1.27 1.27)) (justify right))
     )
-    (property "Footprint" "" (at 150.368 120.65 90)
+    (property "Footprint" "DF_ESC_Footprint_Library:RES-SMD_L7.0-W6.7" (at 150.368 120.65 90)
       (effects (font (size 1.27 1.27)) hide)
     )
@@
       (effects (font (size 1.27 1.27)))
     )
-    (property "Footprint" "" (at 191.77 75.438 90)
+    (property "Footprint" "Resistor_SMD:R_0603_1608Metric_Pad0.98x0.95mm_HandSolder" (at 191.77 75.438 90)
       (effects (font (size 1.27 1.27)) hide)
     )
@@
       (effects (font (size 1.27 1.27)))
     )
-    (property "Footprint" "" (at 60.96 89.408 90)
+    (property "Footprint" "Resistor_SMD:R_0603_1608Metric_Pad0.98x0.95mm_HandSolder" (at 60.96 89.408 90)
       (effects (font (size 1.27 1.27)) hide)
     )
@@
       (effects (font (size 1.27 1.27)) (justify right))
     )
-    (property "Footprint" "" (at 84.328 120.65 90)
+    (property "Footprint" "DF_ESC_Footprint_Library:RES-SMD_L7.0-W6.7" (at 84.328 120.65 90)
       (effects (font (size 1.27 1.27)) hide)
     )
@@
       (effects (font (size 1.27 1.27)) (justify left))
     )
-    (property "Footprint" "" (at 267.97 71.12 0)
+    (property "Footprint" "7461084:WE_7461084" (at 267.97 71.12 0)
       (effects (font (size 1.27 1.27)) hide)
     )
@@
       (effects (font (size 1.27 1.27)))
     )
-    (property "Footprint" "" (at 127 89.408 90)
+    (property "Footprint" "Resistor_SMD:R_0603_1608Metric_Pad0.98x0.95mm_HandSolder" (at 127 89.408 90)
       (effects (font (size 1.27 1.27)) hide)
     )
@@
       (effects (font (size 1.27 1.27)) (justify right))
     )
-    (property "Footprint" "" (at 136.398 95.25 90)
+    (property "Footprint" "Resistor_SMD:R_0603_1608Metric_Pad0.98x0.95mm_HandSolder" (at 136.398 95.25 90)
       (effects (font (size 1.27 1.27)) hide)
     )
@@
       (effects (font (size 1.27 1.27)) (justify left))
     )
-    (property "Footprint" "" (at 57.4548 124.46 0)
+    (property "Footprint" "Capacitor_SMD:C_0603_1608Metric" (at 57.4548 124.46 0)
       (effects (font (size 1.27 1.27)) hide)
     )
@@
       (effects (font (size 1.27 1.27)) (justify left))
     )
-    (property "Footprint" "" (at 267.97 87.63 0)
+    (property "Footprint" "7461084:WE_7461084" (at 267.97 87.63 0)
       (effects (font (size 1.27 1.27)) hide)
     )
@@
       (effects (font (size 1.27 1.27)) (justify left))
     )
-    (property "Footprint" "" (at 85.09 85.09 0)
+    (property "Footprint" "Package_DFN_QFN:PQFN-8-EP_6x5mm_P1.27mm_Generic" (at 85.09 85.09 0)
       (effects (font (size 1.27 1.27)) hide)
     )
@@
       (effects (font (size 1.27 1.27)) (justify left))
     )
-    (property "Footprint" "" (at 123.4948 124.46 0)
+    (property "Footprint" "Capacitor_SMD:C_0603_1608Metric" (at 123.4948 124.46 0)
       (effects (font (size 1.27 1.27)) hide)
     )
@@
       (effects (font (size 1.27 1.27)) (justify right))
     )
-    (property "Footprint" "" (at 148.59 102.87 0)
+    (property "Footprint" "DF_ESC_Footprint_Library:NetTie_SMD_Pad_3.00mm" (at 148.59 102.87 0)
       (effects (font (size 1.27 1.27)) hide)
     )
@@
       (effects (font (size 1.27 1.27)))
     )
-    (property "Footprint" "" (at 199.39 86.36 0)
+    (property "Footprint" "NetTie:NetTie-2_SMD_Pad0.5mm" (at 199.39 86.36 0)
       (effects (font (size 1.27 1.27)) hide)
     )
@@
       (effects (font (size 1.27 1.27)) (justify left))
     )
-    (property "Footprint" "" (at 151.13 85.09 0)
+    (property "Footprint" "Package_DFN_QFN:PQFN-8-EP_6x5mm_P1.27mm_Generic" (at 151.13 85.09 0)
       (effects (font (size 1.27 1.27)) hide)
     )
@@
       (effects (font (size 1.27 1.27)) (justify left))
     )
-    (property "Footprint" "" (at 215.9 71.12 0)
+    (property "Footprint" "Package_DFN_QFN:PQFN-8-EP_6x5mm_P1.27mm_Generic" (at 215.9 71.12 0)
       (effects (font (size 1.27 1.27)) hide)
     )
@@
       (effects (font (size 1.27 1.27)) (justify left))
     )
-    (property "Footprint" "" (at 266.7 54.61 0)
+    (property "Footprint" "7461084:WE_7461084" (at 266.7 54.61 0)
       (effects (font (size 1.27 1.27)) hide)
     )
@@
       (effects (font (size 1.27 1.27)) (justify left))
     )
-    (property "Footprint" "" (at 151.13 59.69 0)
-      (effects (font (size 1.27 1.27)) hide)
-    )
+    (property "Footprint" "Package_DFN_QFN:PQFN-8-EP_6x5mm_P1.27mm_Generic" (at 151.13 59.69 0)
+      (effects (font (size 1.27 1.27)) hide)
+    )
