File: Projects/Fresu/BLDC Motor Controller/Design/rev01/rev01_1/BLDC_Motor Controller/MOSFETS.kicad_sch (KiCad schematic)
At the start: 34 parts, among them J4 7461084, J5 7461084, J6 7461084, Q1 HSBA15810C, Q2 HSBA15810C, Q3 HSBA15810C, Q4 HSBA15810C, Q5 HSBA15810C, Q6 HSBA15810C

Commit message: Update 25
Capturing all updates
Parts:
- added J10: 7461084, 7461084:WE_7461084, symbol ESC_Phase_Connection:7461084
Connections:
- new net: J10.1, J10.2 (1), J10.3 (1), J10.4 (1), J10.5 (1), J10.6 (1), J10.7 (1), J10.8 (1)
Changed lines of the file:
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@@
+	)
+	(symbol
+		(lib_id "ESC_Phase_Connection:7461084")
+		(at 264.16 35.56 0)
+		(unit 1)
+		(exclude_from_sim no)
+		(in_bom yes)
+		(on_board yes)
+		(dnp no)
+		(fields_autoplaced yes)
+		(property "Reference" "J10"
+			(at 270.51 34.2899 0)
+			(effects
+				(font
+					(size 1.27 1.27)
+				)
+				(justify left)
+			)
+		)
+		(property "Value" "7461084"
+			(at 270.51 36.8299 0)
+			(effects
+				(font
+					(size 1.27 1.27)
+				)
+				(justify left)
+			)
+		)
+		(property "Footprint" "7461084:WE_7461084"
+			(at 264.16 35.56 0)
+			(effects
+				(font
+					(size 1.27 1.27)
+				)
+				(justify bottom)
+				(hide yes)
+			)
+		)
+		(property "Datasheet" ""
+			(at 264.16 35.56 0)
+			(effects
+				(font
+					(size 1.27 1.27)
+				)
+				(hide yes)
+			)
+		)
+		(property "Description" ""
+			(at 264.16 35.56 0)
+			(effects
+				(font
+					(size 1.27 1.27)
+				)
+				(hide yes)
+			)
+		)
+		(property "MF" "Wurth Elektronik"
+			(at 264.16 35.56 0)
+			(effects
+				(font
+					(size 1.27 1.27)
+				)
+				(justify bottom)
+				(hide yes)
+			)
+		)
+		(property "MAXIMUM_PACKAGE_HEIGHT" "13.5 mm"
+			(at 264.16 35.56 0)
+			(effects
+				(font
+					(size 1.27 1.27)
+				)
+				(justify bottom)
+				(hide yes)
+			)
+		)
+		(property "Package" "None"
+			(at 264.16 35.56 0)
+			(effects
+				(font
+					(size 1.27 1.27)
+				)
+				(justify bottom)
+				(hide yes)
+			)
+		)
+		(property "Price" "None"
+			(at 264.16 35.56 0)
+			(effects
+				(font
+					(size 1.27 1.27)
+				)
+				(justify bottom)
+				(hide yes)
+			)
+		)
+		(property "Check_prices" "https://www.snapeda.com/parts/7461084/Wurth+Elektronik/view-part/?ref=eda"
+			(at 264.16 35.56 0)
+			(effects
+				(font
+					(size 1.27 1.27)
+				)
+				(justify bottom)
+				(hide yes)
+			)
+		)
+		(property "STANDARD" "Manufacturer Recommendations"
+			(at 264.16 35.56 0)
+			(effects
+				(font
+					(size 1.27 1.27)
+				)
+				(justify bottom)
+				(hide yes)
+			)
+		)
+		(property "PARTREV" "001.002"
+			(at 264.16 35.56 0)
+			(effects
+				(font
+					(size 1.27 1.27)
+				)
+				(justify bottom)
+				(hide yes)
+			)
+		)
+		(property "SnapEDA_Link" "https://www.snapeda.com/parts/7461084/Wurth+Elektronik/view-part/?ref=snap"
+			(at 264.16 35.56 0)
+			(effects
+				(font
+					(size 1.27 1.27)
+				)
+				(justify bottom)
+				(hide yes)
+			)
+		)
+		(property "MP" "7461084"
+			(at 264.16 35.56 0)
+			(effects
+				(font
+					(size 1.27 1.27)
+				)
+				(justify bottom)
+				(hide yes)
+			)
+		)
+		(property "Purchase-URL" "https://www.snapeda.com/api/url_track_click_mouser/?unipart_id=4974952&manufacturer=Wurth Elektronik&part_name=7461084&search_term=None"
+			(at 264.16 35.56 0)
+			(effects
+				(font
+					(size 1.27 1.27)
+				)
+				(justify bottom)
+				(hide yes)
+			)
+		)
+		(property "Description_1" "\n8 Pin Screw Terminal, Power Tap M6 Through Hole\n"
+			(at 264.16 35.56 0)
+			(effects
+				(font
+					(size 1.27 1.27)
+				)
+				(justify bottom)
+				(hide yes)
+			)
+		)
+		(property "MANUFACTURER" "Wurth Electronics"
+			(at 264.16 35.56 0)
+			(effects
+				(font
+					(size 1.27 1.27)
+				)
+				(justify bottom)
+				(hide yes)
+			)
+		)
+		(property "Availability" "In Stock"
+			(at 264.16 35.56 0)
+			(effects
+				(font
+					(size 1.27 1.27)
+				)
+				(justify bottom)
+				(hide yes)
+			)
+		)
+		(property "SNAPEDA_PN" "7461084"
+			(at 264.16 35.56 0)
+			(effects
+				(font
+					(size 1.27 1.27)
+				)
+				(justify bottom)
+				(hide yes)
+			)
+		)
+		(pin "7"
+		)
+		(pin "2"
+		)
+		(pin "6"
+		)
+		(pin "1"
+		)
+		(pin "4"
+		)
+		(pin "5"
+		)
+		(pin "8"
+		)
+		(pin "3"
+		)
+		(instances
+			(project "BLDC_Motor Controller"
+				(path "/e63e39d7-6ac0-4ffd-8aa3-1841a4541b55/6ff318f8-ab62-4d6d-8e81-6536cd3472e5"
+					(reference "J10")
+					(unit 1)
+				)
+			)
+		)
 	)
 	(symbol

Commit message: Update 26
Matched DF's Designators to mine so I can use BOM as is

Updated MFR'ing files

Rev1 Ready for release
Parts:
- removed J10: 7461084, 7461084:WE_7461084, symbol ESC_Phase_Connection:7461084
- renumbered C42 to C45, C43 to C46, J4 to J5, J5 to J6, J6 to J7, R25 to R24, R24 to R25, R31 to R30, R30 to R31, R34 to R32, R37 to R33, R36 to R34, R32 to R35, R33 to R36, R38 to R37, R35 to R38
