File: Projects/Fresu/BLDC Motor Controller/Design/rev01/rev01_1/BLDC_Motor Controller/CAN BUS.kicad_sch (KiCad schematic)
At the start: 0 parts

Commit message: UPDATE 8
COMPLETED CAN SCHEMATIC
Parts:
- added C45, C46: 51p, symbol Device:C
- added C47: 2u2, symbol Device:C
- added D11: ESDCAN24-2BLY, symbol Device:D_TVS_Dual_AAC
- added FL1: 7442275, symbol Device:Filter_EMI_LL_1423
- added J7: Conn_01x04, symbol Connector_Generic:Conn_01x04
- added R39, R40: 10R, symbol Device:R
- added R41: 120R, symbol Device:R
- added R42: 10K, symbol Device:R
- added U3: SN65HVD230, Package_SO:SOIC-8_3.9x4.9mm_P1.27mm, symbol Interface_CAN_LIN:SN65HVD230
Connections:
- new net: R42.2, U3.8 (Rs)
- new net +3V3: C47.1, U3.3 (VCC)
- new net +5V: J7.1 (Pin_1)
- new net CAN_N: FL1.4, U3.6 (CANL)
- new net CAN_P: FL1.3, U3.7 (CANH)
- new net CAN_RX: U3.4 (R)
- new net CAN_TX: U3.1 (D)
- new net C_CAN_N: C46.1, D11.1 (A1), J7.3 (Pin_3), R40.1, R41.1
- new net C_CAN_P: C45.1, D11.2 (A2), J7.2 (Pin_2), R39.1, R41.2
- new net GND: C45.2, C46.2, C47.2, D11.3 (common), J7.4 (Pin_4), R42.1, U3.2 (GND)
- new net R_CAN_N: FL1.1, R40.2
- new net R_CAN_P: FL1.2, R39.2
- no-connect marks 0 -> 1
Other:
- note added: "MODE SLECTION RESISTOR SLEW RATE OF -15 V/uS MORE INFO ON DATASHEET"

Commit message: Update 13
Added:
1) USB Schematic
2) footprints to all parts
Parts:
- removed FL1: 7442275, symbol Device:Filter_EMI_LL_1423
- removed J7: Conn_01x04, symbol Connector_Generic:Conn_01x04
- added FL1: 744227S, DF_ESC_Footprint_Library:FILTER-SMD_4P-L9.2-W6.0-P2.54-TL, symbol DF_ESC_Symbol_Library:744227S
- added U5: S4B-XH-SM4-TB-(LF)(SN), DF_ESC_Footprint_Library:CONN-SMD_S4B-XH-SM4-TB-LF-SN, symbol DF_ESC_Symbol_Library:S4B-XH-SM4-TB-(LF)(SN)
- C45, C46, C47: footprint (none) -> Capacitor_SMD:C_0603_1608Metric
- D11: footprint (none) -> Package_TO_SOT_SMD:TSOT-23
- R39, R40, R41, R42: footprint (none) -> Resistor_SMD:R_0603_1608Metric_Pad0.98x0.95mm_HandSolder
Connections:
- net +5V: now also U5.4
- net CAN_N: now also FL1.4
- net CAN_P: now also FL1.3
- net C_CAN_N: now also U5.2
- net C_CAN_P: now also U5.3
- net GND: now also U5.1
- net R_CAN_N: now also FL1.1
- net R_CAN_P: now also FL1.2
- no-connect marks 1 -> 3

Commit message: Update 15
Fixing some schematic errors

initial layout of larger component complete
Parts:
- renumbered C45 to C44, C46 to C45, C47 to C46, D11 to D9, R41 to R39, R39 to R40, R40 to R41, U5 to U3, U3 to U4

Commit message: Update 20
First layout completed, all tracks laid
Connections:
- net CAN_RX renamed CAN-
- net CAN_TX renamed CAN+
Changed lines of the file:
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@@
+    (stroke (width 0) (type default))
+  )
+  (wire (pts (xy 157.48 115.57) (xy 179.07 115.57))
     (stroke (width 0) (type default))
   )
@@
     (stroke (width 0) (type default))
   )
+  (wire (pts (xy 157.48 113.03) (xy 179.07 113.03))
+    (stroke (width 0) (type default))
+  )
   (wire (pts (xy 107.95 106.68) (xy 102.87 106.68))
     (stroke (width 0) (type default))
@@
   )
   (wire (pts (xy 88.9 120.65) (xy 88.9 127))
-    (stroke (width 0) (type default))
-  )
-  (wire (pts (xy 157.48 113.03) (xy 179.07 113.03))
     (stroke (width 0) (type default))
   )
@@
     (stroke (width 0) (type default))
   )
-  (wire (pts (xy 157.48 115.57) (xy 179.07 115.57))
-    (stroke (width 0) (type default))
-  )
   (text "MODE SLECTION RESISTOR\nSLEW RATE OF -15 V/uS\n\nMORE INFO ON DATASHEET"
     (at 193.04 134.62 0)
     (effects (font (size 1.27 1.27) bold) (justify right bottom))
   )
-  (label "CAN_RX" (at 170.18 115.57 180) (fields_autoplaced)
-    (effects (font (size 1.27 1.27) bold) (justify right bottom))
+  (label "CAN-" (at 157.48 115.57 0) (fields_autoplaced)
+    (effects (font (size 1.27 1.27) bold) (justify left bottom))
   )
   (label "C_CAN_P" (at 58.42 115.57 180) (fields_autoplaced)
@@
     (effects (font (size 1.27 1.27) bold) (justify right bottom))
   )
-  (label "CAN_TX" (at 170.18 113.03 180) (fields_autoplaced)
-    (effects (font (size 1.27 1.27) bold) (justify right bottom))
-  )
   (label "CAN_N" (at 134.62 118.11 180) (fields_autoplaced)
     (effects (font (size 1.27 1.27) bold) (justify right bottom))
   )
-  (global_label "CAN_TX" (shape input) (at 179.07 113.03 0) (fields_autoplaced)
+  (label "CAN+" (at 157.48 113.03 0) (fields_autoplaced)
+    (effects (font (size 1.27 1.27) bold) (justify left bottom))
+  )
+  (global_label "CAN-" (shape input) (at 179.07 115.57 0) (fields_autoplaced)
     (effects (font (size 1.27 1.27) bold) (justify left))
-    (property "Intersheetrefs" "${INTERSHEET_REFS}" (at 189.4601 113.03 0)
+    (property "Intersheetrefs" "${INTERSHEET_REFS}" (at 187.8878 115.57 0)
       (effects (font (size 1.27 1.27)) (justify left) hide)
     )
   )
-  (global_label "CAN_RX" (shape input) (at 179.07 115.57 0) (fields_autoplaced)
+  (global_label "CAN+" (shape input) (at 179.07 113.03 0) (fields_autoplaced)
     (effects (font (size 1.27 1.27) bold) (justify left))
-    (property "Intersheetrefs" "${INTERSHEET_REFS}" (at 189.7625 115.57 0)
+    (property "Intersheetrefs" "${INTERSHEET_REFS}" (at 187.8878 113.03 0)
       (effects (font (size 1.27 1.27)) (justify left) hide)
     )

Commit message: Update 26
Matched DF's Designators to mine so I can use BOM as is

Updated MFR'ing files

Rev1 Ready for release
Parts:
- renumbered C44 to C47, C45 to C48, C46 to C49, D9 to D14, U3 to J8
Changed lines of the file:
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@@
 		(dnp no)
 		(fields_autoplaced yes)
-		(property "Reference" "U3"
-			(at 31.75 115.57 0)
+		(property "Reference" "J8"
+			(at 31.75 115.5699 0)
 			(effects
 				(font
@@
 		)
 		(property "Value" "S4B-XH-SM4-TB-(LF)(SN)"
-			(at 31.75 118.11 0)
+			(at 31.75 118.1099 0)
 			(effects
 				(font
@@
 			(project "BLDC_Motor Controller"
 				(path "/e63e39d7-6ac0-4ffd-8aa3-1841a4541b55/83374fcd-87ee-43a7-8a01-920f2f382f6c"
-					(reference "U3")
+					(reference "J8")
 					(unit 1)
 				)
@@
 		(on_board yes)
 		(dnp no)
-		(property "Reference" "C44"
+		(property "Reference" "C47"
 			(at 82.55 100.33 0)
 			(effects
@@
 			(project "BLDC_Motor Controller"
 				(path "/e63e39d7-6ac0-4ffd-8aa3-1841a4541b55/83374fcd-87ee-43a7-8a01-920f2f382f6c"
-					(reference "C44")
+					(reference "C47")
 					(unit 1)
 				)
@@
 		(on_board yes)
 		(dnp no)
-		(property "Reference" "C46"
+		(property "Reference" "C49"
 			(at 149.86 88.9 0)
 			(effects
@@
 			(project "BLDC_Motor Controller"
 				(path "/e63e39d7-6ac0-4ffd-8aa3-1841a4541b55/83374fcd-87ee-43a7-8a01-920f2f382f6c"
-					(reference "C46")
+					(reference "C49")
 					(unit 1)
 				)
@@
 		(on_board yes)
 		(dnp no)
-		(property "Reference" "C45"
+		(property "Reference" "C48"
 			(at 82.55 133.35 0)
 			(effects
@@
 			(project "BLDC_Motor Controller"
 				(path "/e63e39d7-6ac0-4ffd-8aa3-1841a4541b55/83374fcd-87ee-43a7-8a01-920f2f382f6c"
-					(reference "C45")
+					(reference "C48")
 					(unit 1)
 				)
@@
 		(on_board yes)
 		(dnp no)
-		(property "Reference" "D9"
+		(property "Reference" "D14"
 			(at 74.93 101.6 90)
 			(effects
@@
 			(project "BLDC_Motor Controller"
 				(path "/e63e39d7-6ac0-4ffd-8aa3-1841a4541b55/83374fcd-87ee-43a7-8a01-920f2f382f6c"
-					(reference "D9")
-					(unit 1)
-				)
+					(reference "D14")
+					(unit 1)
+				)
