File: Projects/Fresu/BLDC Motor Controller/Design/rev01/rev01_1/BLDC_Motor Controller/Mechanical.kicad_sch (KiCad schematic)
At the start: 0 parts

Commit message: Update 14
Added 4 mounting holes, imported all components into PCB project, created board outline
Parts:
- added H1, H2, H3, H5: MountingHole_Pad, MountingHole:MountingHole_3.2mm_M3_Pad_Via, symbol Mechanical:MountingHole_Pad
- added R37, R65, R66, R67: 0R, Resistor_SMD:R_0603_1608Metric_Pad0.98x0.95mm_HandSolder, symbol Device:R
Connections:
- new net: H1.1, R65.2
- new net: H5.1, R37.2
- new net: H3.1, R67.2
- new net: H2.1, R66.2
- new net GND: R37.1, R65.1, R66.1, R67.1

Commit message: Update 15
Fixing some schematic errors

initial layout of larger component complete
Parts:
- renumbered H3 to H1, H5 to H2, H2 to H3, H1 to H4, R67 to R51, R37 to R52, R66 to R53, R65 to R54

Commit message: Update 26
Matched DF's Designators to mine so I can use BOM as is

Updated MFR'ing files

Rev1 Ready for release
Parts:
- renumbered R52 to R50, R53 to R52, R54 to R53
Changed lines of the file:
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@@
 		(on_board yes)
 		(dnp no)
-		(property "Reference" "R54"
+		(property "Reference" "R53"
 			(at 71.12 120.65 90)
 			(effects
@@
 			(project "BLDC_Motor Controller"
 				(path "/e63e39d7-6ac0-4ffd-8aa3-1841a4541b55/e37a9f6c-c772-4f76-b91a-38cf2a52ff11"
-					(reference "R54")
+					(reference "R53")
 					(unit 1)
 				)
@@
 		(on_board yes)
 		(dnp no)
-		(property "Reference" "R52"
+		(property "Reference" "R50"
 			(at 45.72 120.65 90)
 			(effects
@@
 			(project "BLDC_Motor Controller"
 				(path "/e63e39d7-6ac0-4ffd-8aa3-1841a4541b55/e37a9f6c-c772-4f76-b91a-38cf2a52ff11"
-					(reference "R52")
+					(reference "R50")
 					(unit 1)
 				)
@@
 		(on_board yes)
 		(dnp no)
-		(property "Reference" "R53"
+		(property "Reference" "R52"
 			(at 69.85 152.4 90)
 			(effects
@@
 			(project "BLDC_Motor Controller"
 				(path "/e63e39d7-6ac0-4ffd-8aa3-1841a4541b55/e37a9f6c-c772-4f76-b91a-38cf2a52ff11"
-					(reference "R53")
-					(unit 1)
-				)
+					(reference "R52")
+					(unit 1)
+				)
